Commit message: 2022-4-28

File: src/model_gazebo/urdf/livox_avia.xacro (robot description, xacro)
@@ -1,5 +1,5 @@
 <?xml version="1.0"?>
 <robot xmlns:xacro="http://ros.org/wiki/xacro">
-  <xacro:property name="M_PI" value="3.1415926"/>
+<xacro:property name="M_PI" value="3.14159"/>
   <xacro:property name="laser_min_range" value="0.1"/>
   <xacro:property name="laser_max_range" value="200.0"/>
@@ -88,5 +88,5 @@
     <xacro:Livox_Mid_gazebo_sensor name="${name}" visualize="${visualize}"/>
   </xacro:macro>
-  <xacro:Livox_AVIA name="livox"/>
+  <xacro:Livox_AVIA name="livox" />
 <xacro:property name="livox_length" value="0.09"/>
 <xacro:property name="livox_x" value="0.1"/>

File: src/model_gazebo/urdf/robot_make.urdf.xacro (robot description, xacro)
@@ -19,4 +19,4 @@
      <xacro:include filename="livox_avia.xacro"/>
      <!-- imu驱动 -->
-     <xacro:include filename="gazebo/imu.xacro"/>
+      <xacro:include filename="gazebo/imu.xacro"/>
 </robot>
